Commit message: Fixed Gazebo UR5 error and robot point to point movement

File: simulation/ur5_description/ur5_and_gripper.urdf (robot description, URDF)
Before this commit: robot ur5, 19 links, 18 joints
Joints:
- removed joint world_joint
- added joint fixed_base: type fixed, parent world, child base_link, origin xyz=0.0 0.0 0.0 rpy=0.0 0.0 0.0

File: simulation/ur5_description/ur5_and_gripper_limited.urdf (robot description, URDF)
Before this commit: robot ur5, 19 links, 18 joints
Joints:
- removed joint world_joint
- added joint fixed_base: type fixed, parent world, child base_link, origin xyz=0.0 0.0 0.0 rpy=0.0 0.0 0.0

File: simulation/ur5_description/ur5_joint_limited_robot.urdf.xacro (robot description, xacro)
@@ -15,9 +15,9 @@
     wrist_3_lower_limit="${-pi}" wrist_3_upper_limit="${pi}"
   />
-  <link name="world" />
-  <joint name="world_joint" type="fixed">
+  <link name="world"/>
+  <joint name="fixed_base" type="fixed">
     <parent link="world"/>
     <child link="base_link"/>
-    <origin rpy="0.0 0.0 -1.57" xyz="1.15 1.0 1.0"/>
+    <origin rpy="0.0 0.0 0.0" xyz="0.0 0.0 0.0"/>
   </joint>
 </robot>

File: simulation/ur5_description/ur5_limited.urdf (robot description, URDF)
Before this commit: robot ur5, 10 links, 9 joints
Joints:
- removed joint world_joint
- added joint fixed_base: type fixed, parent world, child base_link, origin xyz=0.0 0.0 0.0 rpy=0.0 0.0 0.0

File: simulation/ur5_description/ur5_robot.urdf.xacro (robot description, xacro)
@@ -8,9 +8,9 @@
   <!-- arm -->
   <xacro:ur5_robot prefix="" joint_limited="false"/>
-  <link name="world" />
-  <joint name="world_joint" type="fixed">
+  <link name="world"/>
+  <joint name="fixed_base" type="fixed">
     <parent link="world"/>
     <child link="base_link"/>
-    <origin rpy="0.0 0.0 -1.57" xyz="1.15 1.0 1.0"/>
+    <origin rpy="0.0 0.0 0.0" xyz="0.0 0.0 0.0"/>
   </joint>
 </robot>

File: simulation/ur5_description/ur5_test_gripper.urdf (robot description, URDF)
Before this commit: robot ur5, 19 links, 18 joints
Joints:
- removed joint world_joint
- added joint fixed_base: type fixed, parent world, child base_link, origin xyz=0.0 0.0 0.0 rpy=0.0 0.0 0.0
