Commit message: Complete Vacuum Gripper

File: simulation/ur5_description/ur5.urdf.xacro (robot description, xacro)
@@ -299,310 +299,4 @@
       </collision>
     </link>
-    <link name="${prefix}vacuum_gripper">
-      <gravity>0</gravity>
-      <visual>
-        <origin rpy="0 0 0" xyz="0 0 0"/>
-        <geometry>
-          <cylinder radius="0.005" length="0.01"/>
-        </geometry>
-        <material name="transparent">
-          <color rgba="1 0 0 0.5"/>
-        </material>
-      </visual>
-      <inertial>
-        <origin rpy="0 0 0" xyz="0.000000 0.000000 0.000000"/>
-        <mass value="0.0001"/>
-        <inertia ixx="1e-08" ixy="0" ixz="0" iyy="1e-08" iyz="0" izz="1e-08"/>
-      </inertial>
-    </link>
-    <joint name="${prefix}gripper_joint" type="fixed">
-      <parent link="${prefix}ee_link" />
-      <child link="${prefix}vacuum_gripper" />
-      <origin rpy="0 1.5708 0" xyz="0.01 0.0125 0" />
-      <limit effort="50" velocity="50" lower="0" upper="0" />
-      <dynamics damping="0.0" friction="10"/>
-    </joint>
-    <gazebo>
-      <plugin name="gazebo_ros_vacuum_gripper" filename="libgazebo_ros_vacuum_gripper.so">
-        <robotNamespace>/ur5/vacuum_gripper</robotNamespace>
-        <bodyName>vacuum_gripper</bodyName>
-        <topicName>grasping</topicName>
-	    <maxForce>50</maxForce>
-        <maxDistance>0.05</maxDistance>
-        <minDistance>0.01</minDistance>
-      </plugin>
-    </gazebo>
-    <link name="${prefix}vacuum_gripper1">
-      <gravity>0</gravity>
-      <visual>
-        <origin rpy="0 0 0" xyz="0 0 0"/>
-        <geometry>
-          <cylinder radius="0.005" length="0.01"/>
-        </geometry>
-        <material name="transparent">
-          <color rgba="1 0 0 0.5"/>
-        </material>
-      </visual>
-      <inertial>
-        <origin rpy="0 0 0" xyz="0.000000 0.000000 0.000000"/>
-        <mass value="0.0001"/>
-        <inertia ixx="1e-08" ixy="0" ixz="0" iyy="1e-08" iyz="0" izz="1e-08"/>
-      </inertial>
-    </link>
-    <joint name="${prefix}gripper1_joint" type="fixed">
-      <parent link="${prefix}ee_link" />
-      <child link="${prefix}vacuum_gripper1" />
-      <origin rpy="0 1.5708 0" xyz="0.01 -0.0125 0" />
-      <limit effort="50" velocity="50" lower="0" upper="0" />
-      <dynamics damping="0.0" friction="10"/>
-    </joint>
-    <gazebo>
-      <plugin name="gazebo_ros_vacuum_gripper1" filename="libgazebo_ros_vacuum_gripper.so">
-        <robotNamespace>/ur5/vacuum_gripper1</robotNamespace>
-        <bodyName>vacuum_gripper1</bodyName>
-        <topicName>grasping</topicName>
-	    <maxForce>50</maxForce>
-        <maxDistance>0.05</maxDistance>
-        <minDistance>0.01</minDistance>
-      </plugin>
-    </gazebo>
-    <link name="${prefix}vacuum_gripper2">
-      <gravity>0</gravity>
-      <visual>
-        <origin rpy="0 0 0" xyz="0 0 0"/>
-        <geometry>
-          <cylinder radius="0.005" length="0.01"/>
-        </geometry>
-        <material name="transparent">
-          <color rgba="1 0 0 0.5"/>
-        </material>
-      </visual>
-      <inertial>
-        <origin rpy="0 0 0" xyz="0.000000 0.000000 0.000000"/>
-        <mass value="0.0001"/>
-        <inertia ixx="1e-08" ixy="0" ixz="0" iyy="1e-08" iyz="0" izz="1e-08"/>
-      </inertial>
-    </link>
-    <joint name="${prefix}gripper2_joint" type="fixed">
-      <parent link="${prefix}ee_link" />
-      <child link="${prefix}vacuum_gripper2" />
-      <origin rpy="0 1.5708 0" xyz="0.01 0 0.0125" />
-      <limit effort="50" velocity="50" lower="0" upper="0" />
-      <dynamics damping="0.0" friction="10"/>
-    </joint>
-    <gazebo>
-      <plugin name="gazebo_ros_vacuum_gripper2" filename="libgazebo_ros_vacuum_gripper.so">
-        <robotNamespace>/ur5/vacuum_gripper2</robotNamespace>
-        <bodyName>vacuum_gripper2</bodyName>
-        <topicName>grasping</topicName>
-	    <maxForce>50</maxForce>
-        <maxDistance>0.05</maxDistance>
-        <minDistance>0.01</minDistance>
-      </plugin>
-    </gazebo>
-    <link name="${prefix}vacuum_gripper3">
-      <gravity>0</gravity>
-      <visual>
-        <origin rpy="0 0 0" xyz="0 0 0"/>
-        <geometry>
-          <cylinder radius="0.005" length="0.01"/>
-        </geometry>
-        <material name="transparent">
-          <color rgba="1 0 0 0.5"/>
-        </material>
-      </visual>
-      <inertial>
-        <origin rpy="0 0 0" xyz="0.000000 0.000000 0.000000"/>
-        <mass value="0.0001"/>
-        <inertia ixx="1e-08" ixy="0" ixz="0" iyy="1e-08" iyz="0" izz="1e-08"/>
-      </inertial>
-    </link>
-    <joint name="${prefix}gripper3_joint" type="fixed">
-      <parent link="${prefix}ee_link" />
-      <child link="${prefix}vacuum_gripper3" />
-      <origin rpy="0 1.5708 0" xyz="0.01 0 -0.0125" />
-      <limit effort="50" velocity="50" lower="0" upper="0" />
-      <dynamics damping="0.0" friction="10"/>
-    </joint>
-    <gazebo>
-      <plugin name="gazebo_ros_vacuum_gripper3" filename="libgazebo_ros_vacuum_gripper.so">
-        <robotNamespace>/ur5/vacuum_gripper3</robotNamespace>
-        <bodyName>vacuum_gripper3</bodyName>
-        <topicName>grasping</topicName>
-	    <maxForce>50</maxForce>
-        <maxDistance>0.05</maxDistance>
-        <minDistance>0.01</minDistance>
-      </plugin>
-    </gazebo>
-    <link name="${prefix}vacuum_gripper4">
-      <gravity>0</gravity>
-      <visual>
-        <origin rpy="0 0 0" xyz="0 0 0"/>
-        <geometry>
-          <cylinder radius="0.005" length="0.01"/>
-        </geometry>
-        <material name="transparent">
-          <color rgba="1 0 0 0.5"/>
-        </material>
-      </visual>
-      <inertial>
-        <origin rpy="0 0 0" xyz="0.000000 0.000000 0.000000"/>
-        <mass value="0.0001"/>
-        <inertia ixx="1e-08" ixy="0" ixz="0" iyy="1e-08" iyz="0" izz="1e-08"/>
-      </inertial>
-    </link>
-    <joint name="${prefix}gripper4_joint" type="fixed">
-      <parent link="${prefix}ee_link" />
-      <child link="${prefix}vacuum_gripper4" />
-      <origin rpy="0 1.5708 0" xyz="0.01 0 0" />
-      <limit effort="50" velocity="50" lower="0" upper="0" />
-      <dynamics damping="0.0" friction="10"/>
-    </joint>
-    <gazebo>
-      <plugin name="gazebo_ros_vacuum_gripper4" filename="libgazebo_ros_vacuum_gripper.so">
-        <robotNamespace>/ur5/vacuum_gripper4</robotNamespace>
-        <bodyName>vacuum_gripper4</bodyName>
-        <topicName>grasping</topicName>
-	    <maxForce>50</maxForce>
-        <maxDistance>0.05</maxDistance>
-        <minDistance>0.01</minDistance>
-      </plugin>
-    </gazebo>
-    <link name="${prefix}vacuum_gripper5">
-      <gravity>0</gravity>
-      <visual>
-        <origin rpy="0 0 0" xyz="0 0 0"/>
-        <geometry>
-          <cylinder radius="0.005" length="0.01"/>
-        </geometry>
-        <material name="transparent">
-          <color rgba="1 0 0 0.5"/>
-        </material>
-      </visual>
-      <inertial>
-        <origin rpy="0 0 0" xyz="0.000000 0.000000 0.000000"/>
-        <mass value="0.0001"/>
-        <inertia ixx="1e-08" ixy="0" ixz="0" iyy="1e-08" iyz="0" izz="1e-08"/>
-      </inertial>
-    </link>
-    <joint name="${prefix}gripper5_joint" type="fixed">
-      <parent link="${prefix}ee_link" />
-      <child link="${prefix}vacuum_gripper5" />
-      <origin rpy="0 1.5708 0" xyz="0.01 0.0125 0.0125" />
-      <limit effort="50" velocity="50" lower="0" upper="0" />
-      <dynamics damping="0.0" friction="10"/>
-    </joint>
-    <gazebo>
-      <plugin name="gazebo_ros_vacuum_gripper5" filename="libgazebo_ros_vacuum_gripper.so">
-        <robotNamespace>/ur5/vacuum_gripper5</robotNamespace>
-        <bodyName>vacuum_gripper5</bodyName>
-        <topicName>grasping</topicName>
-	    <maxForce>50</maxForce>
-        <maxDistance>0.05</maxDistance>
-        <minDistance>0.01</minDistance>
-      </plugin>
-    </gazebo>
-    <link name="${prefix}vacuum_gripper6">
-      <gravity>0</gravity>
-      <visual>
-        <origin rpy="0 0 0" xyz="0 0 0"/>
-        <geometry>
-          <cylinder radius="0.005" length="0.01"/>
-        </geometry>
-        <material name="transparent">
-          <color rgba="1 0 0 0.5"/>
-        </material>
-      </visual>
-      <inertial>
-        <origin rpy="0 0 0" xyz="0.000000 0.000000 0.000000"/>
-        <mass value="0.0001"/>
-        <inertia ixx="1e-08" ixy="0" ixz="0" iyy="1e-08" iyz="0" izz="1e-08"/>
-      </inertial>
-    </link>
-    <joint name="${prefix}gripper6_joint" type="fixed">
-      <parent link="${prefix}ee_link" />
-      <child link="${prefix}vacuum_gripper6" />
-      <origin rpy="0 1.5708 0" xyz="0.01 -0.0125 0.0125" />
-      <limit effort="50" velocity="50" lower="0" upper="0" />
-      <dynamics damping="0.0" friction="10"/>
-    </joint>
-    <gazebo>
-      <plugin name="gazebo_ros_vacuum_gripper6" filename="libgazebo_ros_vacuum_gripper.so">
-        <robotNamespace>/ur5/vacuum_gripper6</robotNamespace>
-        <bodyName>vacuum_gripper6</bodyName>
-        <topicName>grasping</topicName>
-	    <maxForce>50</maxForce>
-        <maxDistance>0.05</maxDistance>
-        <minDistance>0.01</minDistance>
-      </plugin>
-    </gazebo>
-    <link name="${prefix}vacuum_gripper7">
-      <gravity>0</gravity>
-      <visual>
-        <origin rpy="0 0 0" xyz="0 0 0"/>
-        <geometry>
-          <cylinder radius="0.005" length="0.01"/>
-        </geometry>
-        <material name="transparent">
-          <color rgba="1 0 0 0.5"/>
-        </material>
-      </visual>
-      <inertial>
-        <origin rpy="0 0 0" xyz="0.000000 0.000000 0.000000"/>
-        <mass value="0.0001"/>
-        <inertia ixx="1e-08" ixy="0" ixz="0" iyy="1e-08" iyz="0" izz="1e-08"/>
-      </inertial>
-    </link>
-    <joint name="${prefix}gripper7_joint" type="fixed">
-      <parent link="${prefix}ee_link" />
-      <child link="${prefix}vacuum_gripper7" />
-      <origin rpy="0 1.5708 0" xyz="0.01 0.0125 -0.0125" />
-      <limit effort="50" velocity="50" lower="0" upper="0" />
-      <dynamics damping="0.0" friction="10"/>
-    </joint>
-    <gazebo>
-      <plugin name="gazebo_ros_vacuum_gripper7" filename="libgazebo_ros_vacuum_gripper.so">
-        <robotNamespace>/ur5/vacuum_gripper7</robotNamespace>
-        <bodyName>vacuum_gripper7</bodyName>
-        <topicName>grasping</topicName>
-	    <maxForce>50</maxForce>
-        <maxDistance>0.05</maxDistance>
-        <minDistance>0.01</minDistance>
-      </plugin>
-    </gazebo>
-    <link name="${prefix}vacuum_gripper8">
-      <gravity>0</gravity>
-      <visual>
-        <origin rpy="0 0 0" xyz="0 0 0"/>
-        <geometry>
-          <cylinder radius="0.005" length="0.01"/>
-        </geometry>
-        <material name="transparent">
-          <color rgba="1 0 0 0.5"/>
-        </material>
-      </visual>
-      <inertial>
-        <origin rpy="0 0 0" xyz="0.000000 0.000000 0.000000"/>
-        <mass value="0.0001"/>
-        <inertia ixx="1e-08" ixy="0" ixz="0" iyy="1e-08" iyz="0" izz="1e-08"/>
-      </inertial>
-    </link>
-    <joint name="${prefix}gripper8_joint" type="fixed">
-      <parent link="${prefix}ee_link" />
-      <child link="${prefix}vacuum_gripper8" />
-      <origin rpy="0 1.5708 0" xyz="0.01 -0.0125 -0.0125" />
-      <limit effort="50" velocity="50" lower="0" upper="0" />
-      <dynamics damping="0.0" friction="10"/>
-    </joint>
-    <gazebo>
-      <plugin name="gazebo_ros_vacuum_gripper8" filename="libgazebo_ros_vacuum_gripper.so">
-        <robotNamespace>/ur5/vacuum_gripper8</robotNamespace>
-        <bodyName>vacuum_gripper8</bodyName>
-        <topicName>grasping</topicName>
-	    <maxForce>50</maxForce>
-        <maxDistance>0.05</maxDistance>
-        <minDistance>0.01</minDistance>
-      </plugin>
-    </gazebo>
     <xacro:ur_arm_transmission prefix="${prefix}" />
     <xacro:ur_arm_gazebo prefix="${prefix}" />

File: simulation/ur5_description/ur5_and_gripper.urdf (robot description, URDF)
Before this commit: robot ur5, 19 links, 18 joints
Links:
- removed link vacuum_gripper
- removed link vacuum_gripper1
- removed link vacuum_gripper2
- removed link vacuum_gripper3
- removed link vacuum_gripper4
- removed link vacuum_gripper5
- removed link vacuum_gripper6
- removed link vacuum_gripper7
- removed link vacuum_gripper8
Joints:
- removed joint gripper1_joint
- removed joint gripper2_joint
- removed joint gripper3_joint
- removed joint gripper4_joint
- removed joint gripper5_joint
- removed joint gripper6_joint
- removed joint gripper7_joint
- removed joint gripper8_joint
- removed joint gripper_joint

File: simulation/ur5_description/ur5_and_gripper_limited.urdf (robot description, URDF)
Before this commit: robot ur5, 19 links, 18 joints
Links:
- removed link vacuum_gripper
- removed link vacuum_gripper1
- removed link vacuum_gripper2
- removed link vacuum_gripper3
- removed link vacuum_gripper4
- removed link vacuum_gripper5
- removed link vacuum_gripper6
- removed link vacuum_gripper7
- removed link vacuum_gripper8
Joints:
- removed joint gripper1_joint
- removed joint gripper2_joint
- removed joint gripper3_joint
- removed joint gripper4_joint
- removed joint gripper5_joint
- removed joint gripper6_joint
- removed joint gripper7_joint
- removed joint gripper8_joint
- removed joint gripper_joint
