Commit message: Testing on P52 ThinkPad

File: simulation/ur5_description/ur5_and_gripper_limited.urdf (robot description, URDF)
Before this commit: robot ur5, 10 links, 9 joints
Links:
- link base_link: geometry collision mesh filename=package://semantic_web/simulation/ur5_description/ur5_mesh/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; visual mesh filename=package://semantic_web/simulation/ur5_description/ur5_mesh/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
- link forearm_link: geometry collision mesh filename=package://semantic_web/simulation/ur5_description/ur5_mesh/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; visual mesh filename=package://semantic_web/simulation/ur5_description/ur5_mesh/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
- link shoulder_link: geometry collision mesh filename=package://semantic_web/simulation/ur5_description/ur5_mesh/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; visual mesh filename=package://semantic_web/simulation/ur5_description/ur5_mesh/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
- link upper_arm_link: geometry collision mesh filename=package://semantic_web/simulation/ur5_description/ur5_mesh/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; visual mesh filename=package://semantic_web/simulation/ur5_description/ur5_mesh/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
- link wrist_1_link: geometry collision mesh filename=package://semantic_web/simulation/ur5_description/ur5_mesh/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; visual mesh filename=package://semantic_web/simulation/ur5_description/ur5_mesh/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
- link wrist_2_link: geometry collision mesh filename=package://semantic_web/simulation/ur5_description/ur5_mesh/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; visual mesh filename=package://semantic_web/simulation/ur5_description/ur5_mesh/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
- link wrist_3_link: geometry collision mesh filename=package://semantic_web/simulation/ur5_description/ur5_mesh/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; visual mesh filename=package://semantic_web/simulation/ur5_description/ur5_mesh/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
